Commit message: Correct model

File: urdf/bar_lifting_two_firefly_base.xacro (robot description, xacro)
@@ -12,11 +12,45 @@
   <!-- Creation of UAV_1 -->
   <xacro:firefly_macro
-    namespace="${namespace}">
+    namespace="${namespace}/firefly_1">
+  </xacro:firefly_macro>
+  <!-- Creation of UAV_2 -->
+  <xacro:firefly_macro
+    namespace="${namespace}/firefly_2">
   </xacro:firefly_macro>
   <!-- Attaching the cable to UAV_1 -->
-  <xacro:cable_macro
-    robot_namespace="${namespace}"
-    uav_body_frame="${namespace}/base_link"
-    id_number="1">
-  </xacro:cable_macro>
+  <xacro:payload_macro
+    namespace="${namespace}"
+    uav_1_link="${namespace}/firefly_1/base_link"
+    uav_2_link="${namespace}/firefly_2/base_link" >
+  </xacro:payload_macro>
+  <!-- Adding odometry sensor to the bar -->
+  <xacro:odometry_plugin_macro
+    namespace="${namespace}/bar"
+    odometry_sensor_suffix="_bar"
+    parent_link="${namespace}/bar"
+    pose_topic="ground_truth/pose"
+    pose_with_covariance_topic="ground_truth/pose_with_covariance"
+    position_topic="ground_truth/position"
+    transform_topic="ground_truth/transform"
+    odometry_topic="ground_truth/odometry"
+    parent_frame_id="world"
+    child_frame_id="${namespace}/bar"
+    mass_odometry_sensor="0.00001"
+    measurement_divisor="1"
+    measurement_delay="0"
+    unknown_delay="0.0"
+    noise_normal_position="0 0 0"
+    noise_normal_quaternion="0 0 0"
+    noise_normal_linear_velocity="0 0 0"
+    noise_normal_angular_velocity="0 0 0"
+    noise_uniform_position="0 0 0"
+    noise_uniform_quaternion="0 0 0"
+    noise_uniform_linear_velocity="0 0 0"
+    noise_uniform_angular_velocity="0 0 0"
+    enable_odometry_map="false"
+    odometry_map=""
+    image_scale="">
+    <inertia ixx="0.00001" ixy="0.0" ixz="0.0" iyy="0.00001" iyz="0.0" izz="0.00001" /> <!-- [kg m^2] [kg m^2] [kg m^2] [kg m^2] [kg m^2] [kg m^2] -->
+    <origin xyz="0.0 0.0 0.0" rpy="0.0 0.0 0.0" />
+  </xacro:odometry_plugin_macro>
 </robot>

File: urdf/cables_and_payload.xacro (robot description, xacro)
@@ -17,4 +17,6 @@
   <xacro:property name="z_payload" value="$(arg z_payload)"/> <!-- [m] -->
   <xacro:property name="payload_mass" value="$(arg payload_mass)"/> <!-- [kg] -->
+  <xacro:property name="bar_length" value="1" /> <!-- [m] -->
+  <xacro:property name="bar_radius" value="0.01" /> <!-- [m] -->
   <!-- Macro that creates a cuboid -->
   <xacro:macro name="cuboid_macro" params="x y z mass">
@@ -49,25 +51,66 @@
     </visual>
   </xacro:macro>
-  <!-- Macro that connects a cable to a UAV -->
-  <xacro:macro name="cable_macro"
-    params="robot_namespace uav_body_frame id_number">
-    <!-- ################################################################### -->
-    <!-- ##                             LINKS                             ## -->
-    <!-- ################################################################### -->
-    <!-- This sphere is between payload (root node) and cable -->
-    <link name="${robot_namespace}/aux_pay_${id_number}">
-      <xacro:sphere_macro r="${sphere_radius}" mass="${sphere_mass}"/>
-      <!-- For TESTING purposes:
-      <xacro:cuboid_macro x="0.1" y="0.3" z="0.001" mass="1"/> -->
+  <!-- Macro for uav ball joint -->
+  <xacro:macro name="uav_ball_joint" params="uav_link">
+    <!-- Load of hinge_x, no need for visual or collision for hinge mechanism -->
+    <link name="${uav_link}/load_hinge_x">
+      <inertial>
+        <origin xyz="0 0 0" rpy="0 0 0"/>
+        <mass value="0.01"/>
+        <inertia
+         ixx="0.0001" ixy="0.0" ixz="0.0"
+         iyy="0.0001" iyz="0.0"
+         izz="0.0001"/>
+      </inertial>
     </link>
-    <!-- The CABLE is represented as a cylindrical link -->
-    <link name="${robot_namespace}/cable_${id_number}">
+    <!-- Load of hinge_y, no need for visual or collision for hinge mechanism -->
+    <link name="${uav_link}/load_hinge_y">
       <inertial>
-        <origin xyz="0 0 ${cable_length/2}" rpy="0 0 0"/>
-        <mass value="${cable_mass}"/>
+        <origin xyz="0 0 0" rpy="0 0 0"/>
+        <mass value="0.01"/>
         <inertia
-          ixx="0.0" ixy="0.0" ixz="0.0"
-          iyy="${cable_mass * cable_length * cable_length / 3}" iyz="0.0"
-          izz="${cable_mass * cable_length * cable_length / 3}"/>
+         ixx="0.0001" ixy="0.0" ixz="0.0"
+         iyy="0.0001" iyz="0.0"
+         izz="0.0001"/>
+      </inertial>
+    </link>
+    <!-- Joint bewteen base_link of vehicle and joint that rotates freely around the first body axis-->
+    <joint name="${uav_link}/hinge_y" type="continuous">
+      <parent link="${uav_link}/load_hinge_y"/>
+      <child link="${uav_link}/load_hinge_x"/>
+      <origin xyz="0 0 0" rpy="0 0 0"/>
+      <axis xyz="0 1 0"/>
+    </joint>
+    <!-- Joint bewteen hinge_x and hinge_y -->
+    <!-- Joint that rotates freely around the second body axis of previously rotated reference frame-->
+    <joint name="${uav_link}/hinge_x" type="continuous">
+      <parent link="${uav_link}/load_hinge_x"/>
+      <child link="${uav_link}"/>
+      <origin xyz="0 0 0" rpy="0 0 0"/>
+      <axis xyz="1 0 0"/>
+    </joint>
+  </xacro:macro>
+  <!-- Macro for ball joints in bar -->
+  <xacro:macro name="bar_ball_joint" params="namespace bar_link length">
+    <!-- Load of hinge_x, no need for visual or collision for hinge mechanism -->
+    <link name="${namespace}/load_hinge_y">
+      <inertial>
+        <origin xyz="0 0 0" rpy="0 0 0"/>
+        <mass value="0.01"/>
+        <inertia
+         ixx="0.0001" ixy="0.0" ixz="0.0"
+         iyy="0.0001" iyz="0.0"
+         izz="0.0001"/>
+      </inertial>
+    </link>
+    <!-- Load of hinge_y, no need for visual or collision for hinge mechanism -->
+    <link name="${namespace}/load_hinge_z">
+      <inertial>
+        <origin xyz="0 0 0" rpy="0 0 0"/>
+        <mass value="0.01"/>
+        <inertia
+         ixx="0.0001" ixy="0.0" ixz="0.0"
+         iyy="0.0001" iyz="0.0"
+         izz="0.0001"/>
       </inertial>
       <visual>
@@ -78,61 +121,64 @@
       </visual>
     </link>
-    <!-- This sphere is between cable and uav -->
-    <link name="${robot_namespace}/aux_uav_${id_number}">
-      <xacro:sphere_macro r="${sphere_radius}" mass="${sphere_mass}"/>
-    </link>
-    <!-- ################################################################### -->
-    <!-- ##                            JOINTS                             ## -->
-    <!-- ################################################################### -->
-    <!-- Joint between payload sphere and the cable -->
-    <joint name="${robot_namespace}/joint_sph_cab_${id_number}" type="continuous">
-      <!-- Placing the joint ref frame in the center of the sphere -->
-      <origin xyz="0 0 0" rpy="0 0 0" />
-      <!-- Axis in the CHILD REFERENCE FRAME around which the rotation happens -->
-      <axis xyz="1 0 0" />
-      <parent link="${robot_namespace}/aux_pay_${id_number}" />
-      <child link="${robot_namespace}/cable_${id_number}" />
+    <!-- Joint bewteen base_link of vehicle and joint that rotates freely around the first body axis-->
+    <joint name="${namespace}/hinge_x" type="continuous">
+      <parent link="${bar_link}"/>
+      <child link="${namespace}/load_hinge_y"/>
+      <origin xyz="${length} 0 0" rpy="0 0 0"/>
+      <axis xyz="0 1 0"/>
     </joint>
-    <!-- Joint between the cable and the UAV sphere -->
-    <joint name="${robot_namespace}/joint_cab_sph_${id_number}" type="continuous">
-      <!-- Placing the joint ref frame on the upper end of the cable -->
-      <origin xyz="0 0 ${cable_length}" rpy="0 0 0" />
-      <!-- Axis in the CHILD REFERENCE FRAME around which the rotation happens -->
-      <axis xyz="1 0 0" />
-      <parent link="${robot_namespace}/cable_${id_number}" />
-      <child link="${robot_namespace}/aux_uav_${id_number}" />
-    </joint>
-    <!-- Joint between the UAV sphere amd the UAV-->
-    <joint name="${robot_namespace}/joint_sph_uav_${id_number}" type="continuous">
-      <!-- Placing the joint ref frame in the center of the sphere -->
-      <origin xyz="0 0 0" rpy="0 0 0" />
-      <!-- Axis in the CHILD REFERENCE FRAME around which the rotation happens -->
-      <axis xyz="0 1 0" />
-      <parent link="${robot_namespace}/aux_uav_${id_number}" />
-      <child link="${uav_body_frame}" />
+    <!-- Joint bewteen hinge_x and hinge_y -->
+    <!-- Joint that rotates freely around the second body axis of previously rotated reference frame-->
+    <joint name="${namespace}/hinge_y" type="continuous">
+      <parent link="${namespace}/load_hinge_y"/>
+      <child link="${namespace}/load_hinge_z"/>
+      <origin xyz="0 0 0" rpy="0 0 0"/>
+      <axis xyz="0 0 1"/>
     </joint>
   </xacro:macro>
-  <xacro:macro name="payload_macro" params="link1 link2">
-    <!-- This link represents the payload -->
-    <link name="bar">
-      <xacro:cuboid_macro x="${x_payload}" y="${y_payload}" z="${z_payload}" mass="${payload_mass}"/>
+  <xacro:macro name="payload_macro" params="namespace uav_1_link uav_2_link">
+    <link name="${namespace}/bar">
+      <inertial>
+        <origin xyz="0 0 0" rpy="0 0 0"/>
+        <mass value="${payload_mass}"/>
+        <inertia
+          ixx="0.001" ixy="0.0" ixz="0.0"
+          iyy="${payload_mass * bar_length * bar_length / 12}" iyz="0.0"
+          izz="${payload_mass * bar_length * bar_length / 12}"/>
+      </inertial>
+      <visual>
+        <origin xyz="0 0 0" rpy="-1.570796 0 -1.570796"/>
+        <geometry>
+          <cylinder length="${bar_length}" radius="${bar_radius}"/>
+        </geometry>
+      </visual>
     </link>
-    <!-- Joint connecting to the cable lifterd by the first UAV -->
-    <joint name="bar/joint_sph1" type="continuous">
-      <!-- Placing the joint reference frame on one end of the bar -->
-      <origin xyz="${x_payload/2} 0 ${z_payload/2 + sphere_radius}" rpy="0 0 0" />
-      <!-- Axis in the CHILD REFERENCE FRAME around which the rotation happens -->
-      <axis xyz="0 1 0" />
-      <parent link="bar" />
-      <child link="${link1}" />
+    <xacro:bar_ball_joint
+      namespace="${namespace}/bar_anchor_point_1"
+      bar_link="${namespace}/bar"
+      length="${bar_length/2}">
+    </xacro:bar_ball_joint>
+    <xacro:bar_ball_joint
+      namespace="${namespace}/bar_anchor_point_2"
+      bar_link="${namespace}/bar"
+      length="${-bar_length/2}">
+    </xacro:bar_ball_joint>
+    <xacro:uav_ball_joint
+      uav_link="${uav_1_link}">
+    </xacro:uav_ball_joint>
+    <xacro:uav_ball_joint
+      uav_link="${uav_2_link}">
+    </xacro:uav_ball_joint>
+    <!-- Joint connecting bar anchor to uav -->
+    <joint name="${namespace}/bar_uav_1/joint" type="fixed">
+      <origin xyz="0 0 ${cable_length}" rpy="0 0 0" />
+      <parent link="${namespace}/bar_anchor_point_1/load_hinge_z" />
+      <child link="${uav_1_link}/load_hinge_y" />
     </joint>
-    <!-- Joint connecting to the cable lifterd by the second UAV -->
-    <joint name="bar/joint_sph2" type="continuous">
-      <!-- Placing the joint reference frame on one end of the bar -->
-      <origin xyz="${-x_payload/2} 0 ${z_payload/2 + sphere_radius}" rpy="0 0 0" />
-      <!-- Axis in the CHILD REFERENCE FRAME around which the rotation happens -->
-      <axis xyz="0 1 0" />
-      <parent link="bar" />
-      <child link="${link2}" />
+    <!-- Joint connecting bar anchor to uav -->
+    <joint name="${namespace}/bar_uav_2/joint" type="fixed">
+      <origin xyz="0 0 ${cable_length}" rpy="0 0 0" />
+      <parent link="${namespace}/bar_anchor_point_2/load_hinge_z" />
+      <child link="${uav_2_link}/load_hinge_y" />
     </joint>
   </xacro:macro>
