Commit message: Anchor points do not need to be end points of bar
Also, remove some unnecessary code

File: urdf/cables_and_payload.xacro (robot description, xacro)
@@ -1,8 +1,5 @@
 <?xml version="1.0"?>
 <!--
-  Author: Massimiliano Pandolfo
-  Version 0.7
-  payload_macro now receives two links as input, and acts as root node for the robot tree.
-  With the exception of some minor improvements, this is supposed to be the final version before 1.0.
+  Author:
 -->
 <robot xmlns:xacro="http://ros.org/wiki/xacro">
@@ -10,45 +7,9 @@
   <xacro:property name="cable_length" value="$(arg cable_length)" /> <!-- [m] -->
   <xacro:property name="cable_radius" value="$(arg cable_radius)" /> <!-- [m] -->
-  <xacro:property name="cable_mass" value="$(arg cable_mass)" /> <!-- [kg] -->
-  <xacro:property name="sphere_radius" value="$(arg cable_radius)" /> <!-- [m] -->
-  <xacro:property name="sphere_mass" value="0.001" /> <!-- [kg] -->
-  <xacro:property name="x_payload" value="$(arg x_payload)"/> <!-- [m] -->
-  <xacro:property name="y_payload" value="$(arg y_payload)"/> <!-- [m] -->
-  <xacro:property name="z_payload" value="$(arg z_payload)"/> <!-- [m] -->
   <xacro:property name="payload_mass" value="$(arg payload_mass)"/> <!-- [kg] -->
-  <xacro:property name="bar_length" value="1" /> <!-- [m] -->
-  <xacro:property name="bar_radius" value="0.01" /> <!-- [m] -->
-  <!-- Macro that creates a cuboid -->
-  <xacro:macro name="cuboid_macro" params="x y z mass">
-    <inertial>
-      <origin xyz="0 0 0" rpy="0 0 0"/>
-      <mass value="${mass}"/>
-        <inertia
-        ixx="${mass*(y*y+z*z)/12}" ixy="0.0" ixz="0.0"
-        iyy="${mass*(x*x+z*z)/12}" iyz="0.0"
-        izz="${mass*(y*y+x*x)/12}"/>
-    </inertial>
-    <visual>
-      <geometry>
-        <box size="${x} ${y} ${z}"/>
-      </geometry>
-    </visual>
-  </xacro:macro>
-  <!-- Macro for the auxiliary spheres -->
-  <xacro:macro name="sphere_macro" params="r mass">
-    <inertial>
-      <origin xyz="0 0 0" rpy="0 0 0"/>
-      <mass value="${mass}"/>
-        <inertia
-        ixx="${0.4 * mass * r * r}" ixy="0.0" ixz="0.0"
-        iyy="${0.4 * mass * r * r}" iyz="0.0"
-        izz="${0.4 * mass * r * r}"/>
-    </inertial>
-    <visual>
-      <geometry>
-        <sphere radius="${r}"/>
-      </geometry>
-    </visual>
-  </xacro:macro>
+  <xacro:property name="bar_length" value="$(arg bar_length)" /> <!-- [m] -->
+  <xacro:property name="bar_radius" value="$(arg bar_radius)" /> <!-- [m] -->
+  <xacro:property name="bar_anchor_point1" value="$(arg bar_anchor_point1)" /> <!-- [m] -->
+  <xacro:property name="bar_anchor_point2" value="$(arg bar_anchor_point2)" /> <!-- [m] -->
   <!-- Macro for uav ball joint -->
   <xacro:macro name="uav_ball_joint" params="uav_link">
@@ -157,10 +118,12 @@
       namespace="${namespace}/bar_anchor_point_1"
       bar_link="${namespace}/bar"
-      length="${bar_length/2}">
+      length="${bar_anchor_point1}">
+<!--       length="${bar_length/2}"> -->
     </xacro:bar_ball_joint>
     <xacro:bar_ball_joint
       namespace="${namespace}/bar_anchor_point_2"
       bar_link="${namespace}/bar"
-      length="${-bar_length/2}">
+      length="${bar_anchor_point2}">
+      <!-- length="${-bar_length/2}"> -->
     </xacro:bar_ball_joint>
     <xacro:uav_ball_joint

Commit message: Correct joint axis from z to x
Rotation around z of the link on the bar anchor had no
effect on position of UAV.

Correction:
From joint ${namespace}/hinge_y, around z axis
To joint ${namespace}/bar_hinge_x, around x axis

Some renaming is also done

File: urdf/cables_and_payload.xacro (robot description, xacro)
@@ -36,5 +36,6 @@
       </inertial>
     </link>
-    <!-- Joint bewteen base_link of vehicle and joint that rotates freely around the first body axis-->
+    <!-- Joint bewteen hinge_x and hinge_y -->
+    <!-- Joint that rotates freely around the second body axis-->
     <joint name="${uav_link}/hinge_y" type="continuous">
       <parent link="${uav_link}/load_hinge_y"/>
@@ -43,6 +44,5 @@
       <axis xyz="0 1 0"/>
     </joint>
-    <!-- Joint bewteen hinge_x and hinge_y -->
-    <!-- Joint that rotates freely around the second body axis of previously rotated reference frame-->
+    <!-- Joint bewteen base_link of vehicle and load_hing_x -->
     <joint name="${uav_link}/hinge_x" type="continuous">
       <parent link="${uav_link}/load_hinge_x"/>
@@ -54,5 +54,5 @@
   <!-- Macro for ball joints in bar -->
   <xacro:macro name="bar_ball_joint" params="namespace bar_link length">
-    <!-- Load of hinge_x, no need for visual or collision for hinge mechanism -->
+    <!-- Load of hinge_y: for rotation around y axis of bar -->
     <link name="${namespace}/load_hinge_y">
       <inertial>
@@ -65,6 +65,7 @@
       </inertial>
     </link>
-    <!-- Load of hinge_y, no need for visual or collision for hinge mechanism -->
-    <link name="${namespace}/load_hinge_z">
+    <!-- Load of hinge_x: for rotation around x axis of bar -->
+    <!-- We also use this link to visualize the cable -->
+    <link name="${namespace}/load_hinge_x">
       <inertial>
         <origin xyz="0 0 0" rpy="0 0 0"/>
@@ -82,6 +83,6 @@
       </visual>
     </link>
-    <!-- Joint bewteen base_link of vehicle and joint that rotates freely around the first body axis-->
-    <joint name="${namespace}/hinge_x" type="continuous">
+    <!-- Joint bewteen bar and load_hinge_y located at point in the bar -->
+    <joint name="${namespace}/bar_hinge_y" type="continuous">
       <parent link="${bar_link}"/>
       <child link="${namespace}/load_hinge_y"/>
@@ -89,11 +90,9 @@
       <axis xyz="0 1 0"/>
     </joint>
-    <!-- Joint bewteen hinge_x and hinge_y -->
-    <!-- Joint that rotates freely around the second body axis of previously rotated reference frame-->
-    <joint name="${namespace}/hinge_y" type="continuous">
+    <joint name="${namespace}/bar_hinge_x" type="continuous">
       <parent link="${namespace}/load_hinge_y"/>
-      <child link="${namespace}/load_hinge_z"/>
+      <child link="${namespace}/load_hinge_x"/>
       <origin xyz="0 0 0" rpy="0 0 0"/>
-      <axis xyz="0 0 1"/>
+      <axis xyz="1 0 0"/>
     </joint>
   </xacro:macro>
@@ -109,5 +108,5 @@
       </inertial>
       <visual>
-        <origin xyz="0 0 0" rpy="-1.570796 0 -1.570796"/>
+        <origin xyz="0 0 0" rpy="0 1.570796 0"/>
         <geometry>
           <cylinder length="${bar_length}" radius="${bar_radius}"/>
@@ -136,5 +135,5 @@
     <joint name="${namespace}/bar_uav_1/joint" type="fixed">
       <origin xyz="0 0 ${cable_length}" rpy="0 0 0" />
-      <parent link="${namespace}/bar_anchor_point_1/load_hinge_z" />
+      <parent link="${namespace}/bar_anchor_point_1/load_hinge_x" />
       <child link="${uav_1_link}/load_hinge_y" />
     </joint>
@@ -142,5 +141,5 @@
     <joint name="${namespace}/bar_uav_2/joint" type="fixed">
       <origin xyz="0 0 ${cable_length}" rpy="0 0 0" />
-      <parent link="${namespace}/bar_anchor_point_2/load_hinge_z" />
+      <parent link="${namespace}/bar_anchor_point_2/load_hinge_x" />
       <child link="${uav_2_link}/load_hinge_y" />
     </joint>
